File: Board/project.sch (EAGLE design)
At the start: 21 parts, among them U1 ATMEGA328P_PDIP

Commit message: Updated board.
Parts:
- removed 3V3REGULATOR: V_REG_LD1117VXX, SparkFun-PowerIC:V_REG_LD1117VXX
- added IC1: (no value), SparkFun-PowerIC:V_REG_78XXSIDE
Connections:
- net 3V3: now also IC1.OUT; no longer 3V3REGULATOR.IN
- net BAT_IN: now also IC1.IN; no longer 3V3REGULATOR.GND
- net GND: now also IC1.GND; no longer 3V3REGULATOR.OUT
- net MISO: now also U1.PB4(MISO)
Changed lines of the file:
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@@
 <part name="PROGRAMMER_HEADER" library="SparkFun-Connectors" deviceset="AVR_SPI_PROG2" device="PTH"/>
 <part name="RN42" library="SparkFun-RF" deviceset="XBEE-1" device="B1"/>
-<part name="3V3REGULATOR" library="SparkFun-PowerIC" deviceset="V_REG_LD1117VXX" device=""/>
 <part name="R1" library="SparkFun-Passives" deviceset="RESISTOR" device="AXIAL-0.3" value="10K"/>
 <part name="R2" library="SparkFun-Passives" deviceset="RESISTOR" device="AXIAL-0.3" value="20K"/>
@@
 <part name="GND13" library="SparkFun-Aesthetics" deviceset="GND" device=""/>
 <part name="JP2" library="SparkFun-Passives" deviceset="JUMPER-3-OLD" device="PTH"/>
+<part name="IC1" library="SparkFun-PowerIC" deviceset="V_REG_78XX" device="SIDE"/>
 </parts>
 <sheets>
@@
 <instance part="PROGRAMMER_HEADER" gate="A" x="68.58" y="101.6"/>
 <instance part="RN42" gate="G$1" x="-60.96" y="91.44"/>
-<instance part="3V3REGULATOR" gate="G$1" x="-55.88" y="55.88" rot="R90"/>
 <instance part="R1" gate="G$1" x="-96.52" y="91.44" rot="R90"/>
 <instance part="R2" gate="G$1" x="-88.9" y="91.44" rot="R90"/>
@@
 <instance part="GND13" gate="1" x="30.48" y="10.16"/>
 <instance part="JP2" gate="G$1" x="-7.62" y="30.48"/>
+<instance part="IC1" gate="G$1" x="-55.88" y="63.5"/>
 </instances>
 <busses>
@@
 <wire x1="-53.34" y1="43.18" x2="-43.18" y2="53.34" width="0.1524" layer="91"/>
 <wire x1="-43.18" y1="53.34" x2="-43.18" y2="63.5" width="0.1524" layer="91"/>
-<pinref part="3V3REGULATOR" gate="G$1" pin="OUT"/>
-<wire x1="-43.18" y1="63.5" x2="-55.88" y2="63.5" width="0.1524" layer="91"/>
+<pinref part="IC1" gate="G$1" pin="GND"/>
+<wire x1="-55.88" y1="55.88" x2="-45.72" y2="55.88" width="0.1524" layer="91"/>
+<wire x1="-45.72" y1="55.88" x2="-45.72" y2="63.5" width="0.1524" layer="91"/>
+<wire x1="-45.72" y1="63.5" x2="-43.18" y2="63.5" width="0.1524" layer="91"/>
 </segment>
 </net>
@@
 </segment>
 <segment>
-<pinref part="3V3REGULATOR" gate="G$1" pin="IN"/>
-<wire x1="-55.88" y1="45.72" x2="-55.88" y2="48.26" width="0.1524" layer="91"/>
 <label x="-55.88" y="45.72" size="1.778" layer="95" rot="R90"/>
+<pinref part="IC1" gate="G$1" pin="OUT"/>
+<wire x1="-48.26" y1="63.5" x2="-48.26" y2="53.34" width="0.1524" layer="91"/>
+<wire x1="-48.26" y1="53.34" x2="-55.88" y2="53.34" width="0.1524" layer="91"/>
+<wire x1="-55.88" y1="53.34" x2="-55.88" y2="45.72" width="0.1524" layer="91"/>
 </segment>
 </net>
@@
 <wire x1="-66.04" y1="53.34" x2="-66.04" y2="66.04" width="0.1524" layer="91"/>
 <junction x="-66.04" y="53.34"/>
-<wire x1="-66.04" y1="66.04" x2="-48.26" y2="66.04" width="0.1524" layer="91"/>
-<pinref part="3V3REGULATOR" gate="G$1" pin="GND"/>
-<wire x1="-48.26" y1="66.04" x2="-48.26" y2="55.88" width="0.1524" layer="91"/>
+<pinref part="IC1" gate="G$1" pin="IN"/>
+<wire x1="-63.5" y1="63.5" x2="-63.5" y2="66.04" width="0.1524" layer="91"/>
+<wire x1="-63.5" y1="66.04" x2="-66.04" y2="66.04" width="0.1524" layer="91"/>
 </segment>
 </net>
@@
 <wire x1="60.96" y1="96.52" x2="58.42" y2="96.52" width="0.1524" layer="91"/>
 </segment>
-</net>
+<segment>
+<pinref part="U1" gate="G$1" pin="PB4(MISO)"/>
+<wire x1="30.48" y1="66.04" x2="33.02" y2="66.04" width="0.1524" layer="91"/>
+</segment>
+</net>
